File: gm-board/gm-board.sch (EAGLE design)
At the start: 0 parts

Commit message: done gen bom, almost done coutner
Parts:
- added C10, C21, C22, C23, C6, C8: (no value), passives-7351:CAPACITOR0805-N
- added C11, C19, C2, C20, C3, C4, C5, C7, C9: (no value), passives-7351:CAPACITOR0603-N
- added IC1: ZXCT1109, dtb:ZXCT1109
- added J1: SWD_SHROUD, dtb:SWD_SHROUD
- added J2: HV_GEN, generator-lib:HV_GEN
- added J3: (no value), dtb:JST_2MM_MALE_TH
- added JP1: M05X2SHD, SparkFun-Connectors:M05X2SHD
- added JP2, JP3, JP4: (no value), Mine:M02-HV
- added L6: BEAD, passives-7351:INDUCTOR0603-N
- added R1, R12, R2, R3, R5, R6, R8, R9: (no value), passives-7351:RESISTOR0603-N
- added R10, R11, R13, R18, R4, R7: (no value), passives-7351:RESISTOR1206-N
- added R16, R17: 4k7, passives-7351:RESISTOR0603-N
- added SG2: F/CM12P, buzzer:F/CM12P
- added U$1: STM32F030F4, dtb:STM32F030F4
- added U$2: MCP1700TT, dtb:MCP1700TT
Connections:
- new net +3V3: C19.2, C3.2, C4.2, C5.2, IC1.S+, J1.VCC, JP1.1, R12.P$2, U$1.VDD, U$1.VDDA
- new net CS: JP1.8
- new net GND: C11.1, C20.1, C3.1, C4.1, C5.1, J1.GND1, J1.GND2, J1.GNDD, J2.GND, J2.HV_GND, JP1.2, R16.P$2, R2.P$1, R3.P$1, R5.P$1, R6.P$1, R8.P$1, R9.P$1, SG2.2, U$1.BOOT0, U$1.VSS
- new net HV_CURRENT: C20.2, IC1.OUT, R16.P$1, U$1.PA3
- new net HV_SHDN: J2.SHDN, U$1.PA2
- new net MOSI: JP1.6
- new net N$1: C2.2, JP4.2, R2.P$2
- new net N$16: C10.2, C21.1
- new net N$18: C19.1, IC1.S-, R17.P$2
- new net N$19: C6.1, JP3.1, R7.P$1
- new net N$2: J2.VIN, L6.P$2
- new net N$20: C23.2, C8.2, J2.HV2, R13.P$2, R4.P$2
- new net N$21: R4.P$1, R7.P$2
- new net N$22: C6.2, C8.1
- new net N$23: C22.1, JP2.1, R18.P$1
- new net N$25: R13.P$1, R18.P$2
- new net N$26: C22.2, C23.1
- new net N$3: C10.1, JP4.1, R11.P$1
- new net N$4: R10.P$1, R11.P$2
- new net N$5: C7.2, JP3.2, R5.P$2
- new net N$6: R1.P$1, SG2.1
- new net N$7: C11.2, L6.P$1, R12.P$1, R17.P$1
- new net N$8: C21.2, J2.HV1, R10.P$2
- new net N$9: C9.2, JP2.2, R8.P$2
- new net NRST: J1.NRST, U$1.NRST
- new net SCL: JP1.3, U$1.PA9
- new net SCLK: JP1.5
- new net SDA: JP1.4, U$1.PA10
- new net SWCLK: J1.SWCLK, U$1.PA14
- new net SWDAT: J1.SWDAT, U$1.PA13
- new net TIM14_CH1: R1.P$2, U$1.PA4
- new net TIM16_CH1: C2.1, R3.P$2, U$1.PA6
- new net TIM17_CH1: C7.1, R6.P$2, U$1.PA7
- new net TIM3_CH4: C9.1, R9.P$2, U$1.PB1
Other:
- note added: "Vout = 4700 * 0.004 * V_sense"
