File: gm-board/gm-board.sch (EAGLE design)
At the start: 55 parts, among them IC1 MCP1700TT, IC2 ZXCT1109, IC3 STM32F030F4, J1 HV_GEN-HOLE, J3 SWD_SHROUD, X1 PKM13EPYH, X2 GM-TUBE

Commit message: now to panelize
Parts:
- added LED1, LED2, LED3: (no value), dtb:LEDCHIPLED_0603
- added R19, R20, R21: 220, passives-7351:RESISTOR0603-N
Connections:
- new net LED1: IC3.PA0, LED2.A
- new net LED2: IC3.PA1, LED3.A
- new net LED3: IC3.PF1, LED1.A
- new net N$14: LED1.C, R19.P$1
- new net N$15: LED2.C, R20.P$1
- new net N$17: LED3.C, R21.P$1
- net GND: now also R19.P$2, R20.P$2, R21.P$2
Changed lines of the file:
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@@
 <part name="+3V5" library="supply1" deviceset="+3V3" device=""/>
 <part name="+3V7" library="supply1" deviceset="+3V3" device=""/>
+<part name="LED1" library="dtb" deviceset="LED" device="CHIPLED_0603"/>
+<part name="LED2" library="dtb" deviceset="LED" device="CHIPLED_0603"/>
+<part name="LED3" library="dtb" deviceset="LED" device="CHIPLED_0603"/>
+<part name="R19" library="passives-7351" deviceset="RESISTOR" device="0603-N" value="220"/>
+<part name="R20" library="passives-7351" deviceset="RESISTOR" device="0603-N" value="220"/>
+<part name="R21" library="passives-7351" deviceset="RESISTOR" device="0603-N" value="220"/>
+<part name="GND18" library="supply1" deviceset="GND" device=""/>
+<part name="GND19" library="supply1" deviceset="GND" device=""/>
+<part name="GND20" library="supply1" deviceset="GND" device=""/>
 </parts>
 <sheets>
@@
 <instance part="+3V5" gate="G$1" x="76.2" y="132.08"/>
 <instance part="+3V7" gate="G$1" x="20.32" y="129.54"/>
+<instance part="LED1" gate="G$1" x="109.22" y="10.16"/>
+<instance part="LED2" gate="G$1" x="114.3" y="10.16"/>
+<instance part="LED3" gate="G$1" x="119.38" y="10.16"/>
+<instance part="R19" gate="G$1" x="109.22" y="0" rot="R270"/>
+<instance part="R20" gate="G$1" x="114.3" y="0" rot="R270"/>
+<instance part="R21" gate="G$1" x="119.38" y="0" rot="R270"/>
+<instance part="GND18" gate="1" x="119.38" y="-7.62"/>
+<instance part="GND19" gate="1" x="114.3" y="-7.62"/>
+<instance part="GND20" gate="1" x="109.22" y="-7.62"/>
 </instances>
 <busses>
@@
 <segment>
 <pinref part="R13" gate="G$1" pin="P$2"/>
-<wire x1="111.76" y1="91.44" x2="109.22" y2="88.9" width="0.1524" layer="91"/>
-<wire x1="109.22" y1="88.9" x2="109.22" y2="86.36" width="0.1524" layer="91"/>
+<wire x1="111.76" y1="91.44" x2="109.22" y2="91.44" width="0.1524" layer="91"/>
+<wire x1="109.22" y1="91.44" x2="109.22" y2="86.36" width="0.1524" layer="91"/>
 <pinref part="C13" gate="G$1" pin="2"/>
 <wire x1="109.22" y1="86.36" x2="106.68" y2="86.36" width="0.1524" layer="91"/>
@@
 <pinref part="JP4" gate="G$1" pin="2"/>
 <pinref part="X2" gate="G$1" pin="-"/>
-<wire x1="101.6" y1="93.98" x2="109.22" y2="93.98" width="0.1524" layer="91"/>
-<wire x1="109.22" y1="93.98" x2="109.22" y2="88.9" width="0.1524" layer="91"/>
+<wire x1="101.6" y1="93.98" x2="101.6" y2="91.44" width="0.1524" layer="91"/>
+<wire x1="101.6" y1="91.44" x2="109.22" y2="91.44" width="0.1524" layer="91"/>
 </segment>
 </net>
@@
 <pinref part="GND17" gate="1" pin="GND"/>
 </segment>
+<segment>
+<pinref part="R21" gate="G$1" pin="P$2"/>
+<pinref part="GND18" gate="1" pin="GND"/>
+</segment>
+<segment>
+<pinref part="R20" gate="G$1" pin="P$2"/>
+<pinref part="GND19" gate="1" pin="GND"/>
+</segment>
+<segment>
+<pinref part="R19" gate="G$1" pin="P$2"/>
+<pinref part="GND20" gate="1" pin="GND"/>
+</segment>
 </net>
 <net name="N$5" class="0">
 <segment>
 <pinref part="R11" gate="G$1" pin="P$2"/>
-<wire x1="152.4" y1="91.44" x2="149.86" y2="88.9" width="0.1524" layer="91"/>
-<wire x1="149.86" y1="88.9" x2="149.86" y2="86.36" width="0.1524" layer="91"/>
+<wire x1="152.4" y1="91.44" x2="149.86" y2="91.44" width="0.1524" layer="91"/>
+<wire x1="149.86" y1="91.44" x2="149.86" y2="86.36" width="0.1524" layer="91"/>
 <pinref part="C12" gate="G$1" pin="2"/>
 <wire x1="149.86" y1="86.36" x2="147.32" y2="86.36" width="0.1524" layer="91"/>
@@
 <segment>
 <pinref part="R5" gate="G$1" pin="P$2"/>
-<wire x1="190.5" y1="91.44" x2="187.96" y2="88.9" width="0.1524" layer="91"/>
-<wire x1="187.96" y1="88.9" x2="187.96" y2="86.36" width="0.1524" layer="91"/>
+<wire x1="190.5" y1="91.44" x2="187.96" y2="91.44" width="0.1524" layer="91"/>
+<wire x1="187.96" y1="91.44" x2="187.96" y2="86.36" width="0.1524" layer="91"/>
 <pinref part="C7" gate="G$1" pin="2"/>
 <wire x1="187.96" y1="86.36" x2="185.42" y2="86.36" width="0.1524" layer="91"/>
@@
 </segment>
 </net>
+<net name="N$14" class="0">
+<segment>
+<pinref part="LED1" gate="G$1" pin="C"/>
+<pinref part="R19" gate="G$1" pin="P$1"/>
+</segment>
+</net>
+<net name="N$15" class="0">
+<segment>
+<pinref part="LED2" gate="G$1" pin="C"/>
+<pinref part="R20" gate="G$1" pin="P$1"/>
+</segment>
+</net>
+<net name="N$17" class="0">
+<segment>
+<pinref part="LED3" gate="G$1" pin="C"/>
+<pinref part="R21" gate="G$1" pin="P$1"/>
+</segment>
+</net>
+<net name="LED3" class="0">
+<segment>
+<pinref part="IC3" gate="G$1" pin="PF1"/>
+<wire x1="73.66" y1="15.24" x2="78.74" y2="15.24" width="0.1524" layer="91"/>
+<label x="78.74" y="15.24" size="1.778" layer="95"/>
+</segment>
+<segment>
+<pinref part="LED1" gate="G$1" pin="A"/>
+<wire x1="109.22" y1="12.7" x2="109.22" y2="15.24" width="0.1524" layer="91"/>
+<label x="109.22" y="12.7" size="1.778" layer="95" rot="R90"/>
+</segment>
+</net>
+<net name="LED1" class="0">
+<segment>
+<pinref part="IC3" gate="G$1" pin="PA0"/>
+<wire x1="73.66" y1="68.58" x2="78.74" y2="68.58" width="0.1524" layer="91"/>
+<label x="78.74" y="68.58" size="1.778" layer="95"/>
+</segment>
+<segment>
+<pinref part="LED2" gate="G$1" pin="A"/>
+<wire x1="114.3" y1="12.7" x2="114.3" y2="15.24" width="0.1524" layer="91"/>
+<label x="114.3" y="12.7" size="1.778" layer="95" rot="R90"/>
+</segment>
+</net>
+<net name="LED2" class="0">
+<segment>
+<pinref part="IC3" gate="G$1" pin="PA1"/>
+<wire x1="73.66" y1="66.04" x2="78.74" y2="66.04" width="0.1524" layer="91"/>
+<label x="78.74" y="66.04" size="1.778" layer="95"/>
+</segment>
+<segment>
+<pinref part="LED3" gate="G$1" pin="A"/>
+<wire x1="119.38" y1="12.7" x2="119.38" y2="15.24" width="0.1524" layer="91"/>
+<label x="119.38" y="12.7" size="1.778" layer="95" rot="R90"/>
+</segment>
+</net>
