File: gm-board/gm-board.brd (EAGLE design)
At the start: 56.8 x 31.1 mm, 43 parts, among them IC1 ZXCT1109, J1 SWD_SHROUD, J2 HV_GEN

Commit message: adding part ordering numbers
Parts:
- added C1, C12: 2u2, passives-7351:C0603-N
- C10, C21, C22, C23, C6, C8: value (none) -> 2.2p
- C3: value (none) -> 2u2
- C4, C5: value (none) -> 100n
- R10, R11, R13, R18, R4, R7: value (none) -> 470k
Connections:
- new net N$10: C1.2, J3.1, U$2.3
- net +3V3: now also C12.2, U$2.2
- net GND: now also C1.1, C12.1, J3.2, U$2.1

Commit message: almost done
Parts:
- removed C19: (no value), passives-7351:C0603-N
- removed C21, C22, C23: 2.2p, passives-7351:C0805-N
- removed R17: 4k7, passives-7351:R0603-N
- removed R18: 470k, passives-7351:R1206-N
- removed SG2: F/CM12P, buzzer:F/CM12P
- removed U$2: MCP1700TT, dtb:SOT23
- added C13: (no value), passives-7351:C0603-N
- added C15, C16: 2.2p, passives-7351:C0805-N
- added C17: 100n, passives-7351:C0603-N
- added IC2: ZXCT1109, dtb:SOT23
- added R14, R15: 470k, passives-7351:R1206-N
- added SJ1: JUMPER-PAD-3-2OF3_NC_BY_PASTE, SparkFun-Passives:PAD-JUMPER-3-2OF3_NC_BY_PASTE_YES_SILK_FULL_BOX
- added X1: PKM13EPYH, Mine:PKM13EPYH
- C1, C12, C3: value 2u2 -> (none)
- C11: value (none) -> 2.2p; device passives-7351:C0603-N -> passives-7351:C0805-N
- C2, C9: value (none) -> 2u2
- C4: value 100n -> 2u2
- C5: value 100n -> 2.2p; device passives-7351:C0603-N -> passives-7351:C0805-N
- C8: value 2.2p -> 100n; device passives-7351:C0805-N -> passives-7351:C0603-N
- IC1: value ZXCT1109 -> MCP1700TT
- J1: value SWD_SHROUD -> HV_GEN-HOLE; device dtb:SWD_PTH_SHROUD -> generator-lib:BRD-LAYOUT2
- J2: value HV_GEN -> (none); device generator-lib:BRD-LAYOUT -> dtb:JST-2-TH
- J3: value (none) -> SWD_SHROUD; device dtb:JST-2-TH -> dtb:SWD_PTH_SHROUD
- JP1: value M05X2SHD -> (none); device SparkFun-Connectors:2X5-SHROUDED -> Mine:M03-HV
- JP2: value (none) -> M05X2SHD; device Mine:M03-HV -> SparkFun-Connectors:2X5-SHROUDED
- R1, R6: value (none) -> 4k7
- R11, R13, R7: value 470k -> (none); device passives-7351:R1206-N -> passives-7351:R0603-N
- R16: value 4k7 -> (none)
- R3, R9: value (none) -> 470k; device passives-7351:R0603-N -> passives-7351:R1206-N
- moved C1 63.2 mm to (48.0, 23.0), turned to 90 degrees
- moved C11 39.5 mm to (10.3, 11.3), turned to 180 degrees
- moved C12 36.0 mm to (21.8, 10.2), turned to 180 degrees
- moved J2 31.8 mm to (22.2, 23.5), turned to 0 degrees
- moved R2 28.4 mm to (46.1, 23.0), turned to 270 degrees
- moved J1 27.7 mm to (54.0, 25.4), turned to 180 degrees
- moved R16 25.8 mm to (21.8, 4.45), turned to 0 degrees
- moved JP1 24.8 mm to (12.7, 15.9)
- moved JP2 24.8 mm to (37.3, 13.3)
- moved C5 23.2 mm to (6.73, 17.4), turned to 180 degrees
- moved R3 21.8 mm to (6.22, 19.7), turned to 180 degrees
- moved R6 21.7 mm to (42.9, 19.3), turned to 90 degrees
- moved C8 21.5 mm to (27.9, 13.7)
- moved R12 20.0 mm to (31.8, 9.02), turned to 90 degrees
- moved R13 19.4 mm to (21.8, 8.26)
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- renumbered C20 to C14, L6 to L1, U$1 to IC3
Connections:
- removed net N$10: C1.2, J3.1, U$2.3
- new net N$11: C3.2, IC2.2, R2.2, SJ1.2
- new net VIN: C4.2, IC1.3, J2.1, SJ1.1
- net +3V3: now also C17.2, C2.2, C8.2, C9.2, J3.1, JP2.1, SJ1.3; no longer C12.2, C19.2, C3.2, C4.2, C5.2, J1.1, JP1.1, R12.2, U$2.2
- net CS: now also JP2.8; no longer JP1.8
- net GND: now also C17.1, C2.1, C8.1, C9.1, IC1.1, J1.GND_HV, J1.GND_LV, J2.2, J3.3, J3.5, J3.9, JP2.2, R11.1, R13.1, R16.1, R6.2, R7.1, X1.2; no longer C11.1, C12.1, C3.1, C5.1, J1.3, J1.5, J1.9, J2.GND_HV, J2.GND_LV, J3.2, JP1.2, R16.2, R2.1, R3.1, R6.1, R9.1, SG2.-, U$2.1
- net HV_CURRENT: now also IC2.1, R6.1; no longer IC1.1, R16.1
- net HV_SHDN: now also J1.SHDN; no longer J2.SHDN
- net MOSI: now also JP2.6; no longer JP1.6
- net N$1: now also C13.2, R13.2; no longer C2.2, R2.2
- net N$16: now also C15.1, C16.2; no longer C10.2, C21.1
- net N$18: now also C3.1, IC2.3, R1.2; no longer C19.1, IC1.3, R17.2
- net N$19: now also C11.1, R10.1; no longer C6.1, R7.1
- net N$2: now also J1.VIN; no longer J2.VIN
- net N$20: now also C10.2, C5.2, J1.HV2, R3.2, R9.2; no longer C23.2, C8.2, J2.HV2, R13.2, R4.2
- net N$21: now also R10.2, R9.1; no longer R4.1, R7.2
- net N$22: now also C10.1, C11.2; no longer C6.2, C8.1
- net N$23: now also C6.1, JP1.1, R4.1; no longer C22.1, JP2.1, R18.1
- net N$25: now also R3.1, R4.2; no longer R13.1, R18.2
- net N$26: now also C5.1, C6.2; no longer C22.2, C23.1
- net N$3: now also C16.1, R15.1; no longer C10.1, R11.1
- net N$4: now also R14.1, R15.2; no longer R10.1, R11.2
- net N$5: now also C12.2, R11.2; no longer C7.2, R5.2
- net N$6: now also R12.1, X1.1; no longer R1.1, SG2.+
- net N$7: now also C1.2, R1.1, R2.1; no longer C11.2, R12.1, R17.1
- net N$8: now also C15.2, J1.HV1, R14.2; no longer C21.2, J2.HV1, R10.2
- net N$9: now also C7.2, JP1.3, R5.2; no longer C9.2, JP2.3, R8.2
- net NRST: now also J3.10; no longer J1.10
- net SCL: now also JP2.3; no longer JP1.3
- net SCLK: now also JP2.5; no longer JP1.5
- net SDA: now also JP2.4; no longer JP1.4
- net SWCLK: now also J3.4; no longer J1.4
- net SWDAT: now also J3.2; no longer J1.2
- net TIM14_CH1: now also R12.2; no longer R1.2
- net TIM16_CH1: now also C13.1, R16.2; no longer C2.1, R3.2
- net TIM17_CH1: now also C12.1, R8.2; no longer C7.1, R6.2
- net TIM3_CH4: now also C7.1, R7.2; no longer C9.1, R9.2
Routing:
- net +3V3: track 55.5 -> 79.6 mm, vias 2 -> 6
- net NRST: track 15.2 -> 23.3 mm, vias 0 -> 2
- net VIN: track 0.00 -> 6.73 mm
- net GND: track 32.3 -> 38.3 mm
- net N$11: track 0.00 -> 4.61 mm
- net N$7: track 4.19 -> 6.00 mm
- net N$8: track 33.6 -> 32.3 mm
- net N$6: track 19.0 -> 20.2 mm
- net HV_SHDN: track 41.7 -> 40.8 mm
- net SWDAT: track 8.72 -> 7.83 mm
- net TIM14_CH1: track 5.22 -> 4.68 mm
Other:
- outline, holes or cut-outs redrawn

Commit message: gettuing there...
Parts:
- added R17, R18: (no value), passives-7351:R0603-N
- added TP1, TP2, TP3, TP4, TP5, TP6: TPTP09R, testpad:TP09R
- added X2: GM-TUBE, Mine:GM-TUBE
- J2: device dtb:JST-2-TH -> dtb:JST-2-TH-NOTEXT
- moved J1 55.2 mm to (5.00, 0.00), turned to 0 degrees
- moved R3 48.6 mm to (52.8, 5.71), turned to 0 degrees
- moved C15 48.1 mm to (52.4, 20.1), turned to 0 degrees
- moved R14 47.7 mm to (52.8, 17.9), turned to 0 degrees
- moved R9 46.6 mm to (52.8, 11.8), turned to 0 degrees
- moved C5 46.5 mm to (52.2, 8.00), turned to 0 degrees
- moved C10 45.9 mm to (52.4, 14.1), turned to 0 degrees
- moved L1 45.7 mm to (9.06, 2.41), turned to 90 degrees
- moved C1 42.4 mm to (11.0, 2.41), turned to 270 degrees
- moved C16 41.4 mm to (48.8, 20.1), turned to 0 degrees
- moved R4 40.1 mm to (48.3, 5.71), turned to 0 degrees
- moved C6 39.5 mm to (48.7, 8.00), turned to 0 degrees
- moved R2 39.1 mm to (12.9, 2.41), turned to 90 degrees
- moved R15 39.1 mm to (48.3, 17.9), turned to 0 degrees
- moved C11 38.5 mm to (48.7, 14.1), turned to 0 degrees
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Connections:
- new net N$10: J1.HV3, TP1.TP
- new net N$12: J1.HV2, TP2.TP, TP6.TP
- new net N$13: J1.HV1, TP3.TP
- net +3V3: now also R17.2, R18.2
- net N$1: now also X2.B1, X2.B2
- net N$20: now also TP4.TP; no longer J1.HV2
- net N$3: now also X2.A1, X2.A2
- net N$8: now also TP5.TP; no longer J1.HV1
- net SCL: now also R17.1
- net SDA: now also R18.1
Routing:
- net N$1: track 4.45 -> 51.7 mm
- net N$3: track 5.34 -> 21.2 mm
- net VIN: track 6.73 -> 18.9 mm, vias 0 -> 1
- net N$11: track 4.61 -> 16.3 mm, vias 0 -> 1
- net SCL: track 13.0 -> 21.2 mm
- net HV_CURRENT: track 44.5 -> 36.7 mm
- net +3V3: track 79.6 -> 86.0 mm, vias 6 -> 5
- net N$8: track 32.3 -> 27.3 mm, vias 0 -> 1
- net GND: track 38.3 -> 42.8 mm, vias 12 -> 13
- net N$12: track 0.00 -> 3.27 mm
- net TIM17_CH1: track 11.7 -> 9.33 mm
- net N$10: track 0.00 -> 2.19 mm
- net SWCLK: track 12.2 -> 10.7 mm
- net HV_SHDN: track 40.8 -> 39.4 mm
- net N$13: track 0.00 -> 1.40 mm
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Other:
- board size 56.8 x 31.1 mm -> 59.5 x 31.5 mm
- board text removed: "check polarity"

Commit message: now to panelize
Parts:
- added LED1, LED2, LED3: (no value), dtb:CHIPLED_0603
- added R19, R20, R21: 220, passives-7351:R0603-N
- moved C14 21.6 mm to (10.1, 6.22)
- moved JP2 1.78 mm to (21.6, 10.3)
- moved TP3 0.52 mm to (44.7, 2.79)
- moved TP5 0.46 mm to (47.2, 3.68)
- moved R12 0.38 mm to (27.2, 16.8)
- moved X1 0.35 mm to (10.1, 14.4)
- moved C17 0.33 mm to (33.3, 21.0)
Connections:
- new net LED1: IC3.6, LED2.A
- new net LED2: IC3.7, LED3.A
- new net LED3: IC3.3, LED1.A
- new net N$14: LED1.C, R19.1
- new net N$15: LED2.C, R20.1
- new net N$17: LED3.C, R21.1
- net GND: now also R19.2, R20.2, R21.2
Routing:
- net LED2: track 0.00 -> 15.4 mm
- net LED1: track 0.00 -> 12.7 mm
- net N$15: track 0.00 -> 12.6 mm, vias 0 -> 2
- net N$17: track 0.00 -> 12.5 mm
- net LED3: track 0.00 -> 11.6 mm
- net N$14: track 0.00 -> 9.16 mm, vias 0 -> 2
- net HV_CURRENT: track 36.7 -> 41.5 mm, vias 0 -> 2
- net GND: track 42.8 -> 45.7 mm, vias 13 -> 14
- net N$6: track 20.2 -> 17.8 mm
- net SDA: track 17.8 -> 19.6 mm
- net N$1: track 51.7 -> 51.1 mm
- net +3V3: track 86.0 -> 85.4 mm, vias 5 -> 3
Other:
- outline, holes or cut-outs redrawn
- board text added: "+"
- board text added: "-"
- board text added: "Feb 2016"
- board text added: "Matt Brejza"

Commit message: about to panelize
Parts:
- moved TP5 3.70 mm to (50.4, 5.59)
- moved TP6 2.05 mm to (48.6, 3.05)
- moved C7 1.91 mm to (37.1, 7.62)
- moved R7 1.91 mm to (37.1, 9.53)
- moved R17 0.92 mm to (16.1, 9.14), turned to 270 degrees
- moved TP2 0.57 mm to (49.8, 2.41)
- moved TP3 0.40 mm to (44.3, 2.92)
Routing:
- net N$8: track 27.3 -> 23.5 mm
- net N$9: track 6.80 -> 4.16 mm
- net +3V3: track 85.4 -> 84.8 mm
- net GND: track 45.7 -> 45.1 mm, vias 14 -> 15
Other:
- outline, holes or cut-outs redrawn
